Commit message: Refactor into many packages

File: apc_description/data/models/lwa4d_sdh/urdf/lwa4d_sdh.urdf (robot description, URDF)
Before this commit: robot lwa4d, 21 links, 20 joints
Links:
- link L1_link: geometry collision mesh filename=package://apc_ros/data/models/lwa4d/meshes/arm_1_link.dae; visual mesh filename=package://apc_ros/data/models/lwa4d/meshes/arm_1_link.dae
- link L2_link: geometry collision mesh filename=package://apc_ros/data/models/lwa4d/meshes/arm_2_link.dae; visual mesh filename=package://apc_ros/data/models/lwa4d/meshes/arm_2_link.dae
- link L3_link: geometry collision mesh filename=package://apc_ros/data/models/lwa4d/meshes/arm_3_link.dae; visual mesh filename=package://apc_ros/data/models/lwa4d/meshes/arm_3_link.dae
- link L4_link: geometry collision mesh filename=package://apc_ros/data/models/lwa4d/meshes/arm_4_link.dae; visual mesh filename=package://apc_ros/data/models/lwa4d/meshes/arm_4_link.dae
- link L5_link: geometry collision mesh filename=package://apc_ros/data/models/lwa4d/meshes/arm_5_link.dae; visual mesh filename=package://apc_ros/data/models/lwa4d/meshes/arm_5_link.dae
- link L6_link: geometry collision mesh filename=package://apc_ros/data/models/lwa4d/meshes/arm_6_link.dae; visual mesh filename=package://apc_ros/data/models/lwa4d/meshes/arm_6_link.dae
- link L7_link: geometry collision mesh filename=package://apc_ros/data/models/lwa4d/meshes/arm_7_link.dae; visual mesh filename=package://apc_ros/data/models/lwa4d/meshes/arm_7_link.dae
Joints:
- joint finger_21_joint: origin xyz=0.01905 -0.033 0.0745 rpy=0 0 3.14159265 -> xyz=-0.033 -0.01905 0.0745 rpy=0 0 1.5708
- joint knuckle_joint: origin xyz=0.01905 0.033 0.0745 rpy=0 0 3.14159265 -> xyz= 0.033 -0.01905 0.0745 rpy=0 0 1.5708
- joint thumb_1_joint: origin xyz=-0.03811 0 0.0745  rpy=0 0 0 -> xyz=0.0 0.03811 0.0745  rpy=0 0 -1.5708
