Commit message: Send joint trajectories over ACH to robot arms

File: apc_description/urdf/sdh/sdh.urdf.xacro (robot description, xacro)
@@ -49,5 +49,5 @@
 		<!-- joint between sdh_palm_link and sdh_finger_11_link -->
 		<joint name="${name}_knuckle_joint" type="revolute">
-			<origin xyz="0.033 -0.01905 0.0745" rpy="0 0 1.5708" />
+			<origin xyz="-0.033 -0.01905 0.0745" rpy="0 0 ${-M_PI/2}" />
 			<parent link="${name}_palm_link"/>
 			<child link="${name}_finger_11_link"/>
@@ -138,5 +138,5 @@
 		<joint name="${name}_finger_21_joint" type="revolute">
 			<mimic joint="${name}_knuckle_joint" multiplier="1" offset="0"/>
-			<origin xyz="-0.033 -0.01905 0.0745" rpy="0 0 1.5708" />
+			<origin xyz="0.033 -0.01905 0.0745" rpy="0 0 ${-M_PI/2}" />
 			<parent link="${name}_palm_link"/>
 			<child link="${name}_finger_21_link"/>

Commit message: Fix finger joint orientation in sdh.urdf.xacro

File: apc_description/urdf/sdh/sdh.urdf.xacro (robot description, xacro)
@@ -49,5 +49,6 @@
 		<!-- joint between sdh_palm_link and sdh_finger_11_link -->
 		<joint name="${name}_knuckle_joint" type="revolute">
-			<origin xyz="-0.033 -0.01905 0.0745" rpy="0 0 ${-M_PI/2}" />
+			<!-- <origin xyz="-0.033 -0.01905 0.0745" rpy="0 0 ${-M_PI/2}" /> -->
+			<origin xyz="0.033 -0.01905 0.0745" rpy="0 0 ${M_PI/2}" />
 			<parent link="${name}_palm_link"/>
 			<child link="${name}_finger_11_link"/>
@@ -138,5 +139,5 @@
 		<joint name="${name}_finger_21_joint" type="revolute">
 			<mimic joint="${name}_knuckle_joint" multiplier="1" offset="0"/>
-			<origin xyz="0.033 -0.01905 0.0745" rpy="0 0 ${-M_PI/2}" />
+			<origin xyz="-0.033 -0.01905 0.0745" rpy="0 0 ${M_PI/2}" />
 			<parent link="${name}_palm_link"/>
 			<child link="${name}_finger_21_link"/>
