Commit message: urdf: patch moveit with new crichton model

File: apc_description/urdf/lwa4d/lwa4d.urdf.xacro (robot description, xacro)
@@ -71,5 +71,5 @@
 				<origin xyz="0 0 0" rpy="0 0 0" />
 				<geometry>
-					<mesh filename="package://apc_description/lwa4d/meshes/arm_2_link.dae" />
+					<mesh filename="package://apc_description/meshes/lwa4d/arm_2_link.dae" />
 				</geometry>
 				<material name="Schunk_Black" />
@@ -188,5 +188,5 @@
 		</link>
 	    <!-- J0 -->
-	    <joint name="${name}_0_joint" type="floating" >
+	    <joint name="${name}_0_joint" type="fixed" >
             <xacro:insert_block name="origin"/>
 		    <parent link="${parent}" />

File: apc_description/urdf/lwa4d_torso/lwa4d_torso.urdf.xacro (robot description, xacro)
@@ -2,9 +2,4 @@
 <robot xmlns:xacro="http://www.ros.org/wiki/xacro">
 	<xacro:macro name="schunk_lwa4d_torso" params="parent name *origin">
-		<joint name="${name}_base_joint" type="fixed">
-			<xacro:insert_block name="origin"/>
-			<parent link="${parent}" />
-			<child  link="${name}_vertical_support" />
-		</joint>
 		<link name="${name}_vertical_support">
 			<inertial>
@@ -14,11 +9,35 @@
 			</inertial>
 			<visual>
+				<origin xyz="-0.45 -0.45 0.0" rpy="0 0 0"/>
 				<geometry>
-					<mesh filename="package://apc_description/meshes/vertical_support.dae" scale="1 1 1" />
+					<mesh filename="package://apc_description/meshes/lwa4d_torso/vertical_support.dae" scale="1 1 1" />
+				</geometry>
+			</visual>
+			<collision>
+				<origin xyz="-0.45 -0.45 0.0" rpy="0 0 0"/>
+				<geometry>
+					<mesh filename="package://apc_description/meshes/lwa4d_torso/vertical_support.dae" scale="1 1 1" />
+				</geometry>
+			</collision>
+		</link>
+		<joint name="${name}_base_joint" type="fixed">
+			<xacro:insert_block name="origin"/>
+			<parent link="${parent}" />
+			<child  link="${name}_vertical_support" />
+		</joint>
+		<link name="${name}_middle_support">
+			<inertial>
+				<origin xyz="0.0 0.0 0.0" rpy="0 0 0"/>
+				<mass value="5.0"/>
+				<inertia ixx="1" ixy="0.0" ixz="0.0" iyy="1" iyz="0.0" izz="1" />
+			</inertial>
+			<visual>
+				<geometry>
+					<mesh filename="package://apc_description/meshes/lwa4d_torso/middle_support.dae" scale="1 1 1" />
 				</geometry>
 			</visual>
 			<collision>
 				<geometry>
-					<mesh filename="package://apc_description/meshes/vertical_support.dae" scale="1 1 1" />
+					<mesh filename="package://apc_description/meshes/lwa4d_torso/middle_support.dae" scale="1 1 1" />
 				</geometry>
 			</collision>
@@ -30,21 +49,4 @@
 			<child  link="${name}_middle_support" />
 		</joint>
-		<link name="${name}_middle_support">
-			<inertial>
-				<origin xyz="0.0 0.0 0.0" rpy="0 0 0"/>
-				<mass value="5.0"/>
-				<inertia ixx="1" ixy="0.0" ixz="0.0" iyy="1" iyz="0.0" izz="1" />
-			</inertial>
-			<visual>
-				<geometry>
-					<mesh filename="package://apc_description/meshes/middle_support.dae" scale="1 1 1" />
-				</geometry>
-			</visual>
-			<collision>
-				<geometry>
-					<mesh filename="package://apc_description/meshes/middle_support.dae" scale="1 1 1" />
-				</geometry>
-			</collision>
-		</link>
 	</xacro:macro>
 </robot>

File: apc_description/urdf/sdh/sdh.urdf.xacro (robot description, xacro)
@@ -5,6 +5,6 @@
 	<xacro:macro name="schunk_sdh" params="parent name *origin">
 		<!-- joint between arm_7_link and sdh_palm_link -->
-		<joint name="${name}_palm_joint" type="floating" >
-			<origin xyz="0 0 0" rpy="0 0 0"/>
+		<joint name="${name}_palm_joint" type="fixed" >
+			<origin xyz="0 0 0" rpy="0 ${M_PI} ${- M_PI / 6}"/>
 			<parent link="${parent}" />
 			<child link="${name}_palm_link" />
@@ -137,5 +137,5 @@
 		<!-- joint between sdh_palm_link and sdh_finger_21_link -->
 		<joint name="${name}_finger_21_joint" type="revolute">
-			<mimic joint="knuckle_joint" multiplier="1" offset="0"/>
+			<mimic joint="${name}_knuckle_joint" multiplier="1" offset="0"/>
 			<origin xyz="-0.033 -0.01905 0.0745" rpy="0 0 1.5708" />
 			<parent link="${name}_palm_link"/>

Commit message: Reduce joint limits on crichton model by PI

File: apc_description/urdf/lwa4d/lwa4d.urdf.xacro (robot description, xacro)
@@ -201,5 +201,5 @@
 			<axis xyz="0 0 1"/>
 			<dynamics damping="10" />
-			<limit effort="370" velocity="2.0" lower="-6.2831853" upper="6.2831853"/>
+			<limit effort="370" velocity="2.0" lower="-3.14" upper="3.14"/>
 		</joint>
 	    <!-- J2 -->
@@ -219,5 +219,5 @@
 			<axis xyz="0 0 1"/>
 			<dynamics damping="5" />
-			<limit effort="176" velocity="2.0" lower="-6.2831853" upper="6.2831853"/>
+			<limit effort="176" velocity="2.0" lower="-3.14" upper="3.14"/>
 		</joint>
 		<!-- J4 -->
@@ -237,5 +237,5 @@
 			<axis xyz="0 0 1" />
 			<dynamics damping="5" />
-			<limit effort="41.6" velocity="2.0" lower="-6.2831853" upper="6.2831853" />
+			<limit effort="41.6" velocity="2.0" lower="-3.14" upper="3.14" />
 		</joint>
 		<!-- J6 -->
@@ -255,5 +255,5 @@
 			<axis xyz="0 0 -1" />
 			<dynamics damping="5" />
-			<limit effort="9.6" velocity="2.0" lower="-6.2831853" upper="6.2831853" />
+			<limit effort="9.6" velocity="2.0" lower="-3.14" upper="3.14" />
 		</joint>
         <!-- extensions -->
