Commit message: Change PI constant in URDF to a higher precision

File: apc_description/urdf/lwa4d/lwa4d.xacro (robot description, xacro)
@@ -196,5 +196,5 @@
 		<joint name="${name}_1_joint" type="revolute">
 			<!-- <origin xyz="0 0.1375 0" rpy="1.57 3.1416 0"/> -->
-			<origin xyz="0 0.12 0" rpy="1.57 3.1416 0"/>
+			<origin xyz="0 0.12 0" rpy="${M_PI / 2.0} ${M_PI} 0"/>
 			<parent link="${name}_0_link"/>
 			<child link="${name}_1_link"/>
@@ -205,5 +205,5 @@
 	    <!-- J2 -->
 		<joint name="${name}_2_joint" type="revolute">
-			<origin xyz="0 0 -0.18" rpy="-1.57 0 0"/>
+			<origin xyz="0 0 -0.18" rpy="${ -M_PI / 2.0} 0 0"/>
 			<parent link="${name}_1_link"/>
 			<child link="${name}_2_link"/>
@@ -214,5 +214,5 @@
 		<!-- J3-->
 		<joint name="${name}_3_joint" type="revolute">
-			<origin xyz="0 0 0" rpy="1.57 0 0"/>
+			<origin xyz="0 0 0" rpy="${ M_PI / 2.0 } 0 0"/>
 			<parent link="${name}_2_link"/>
 			<child link="${name}_3_link"/>
@@ -223,5 +223,5 @@
 		<!-- J4 -->
 		<joint name="${name}_4_joint" type="revolute">
-			<origin xyz="0 0 -0.328" rpy="-1.57 0 0"/>
+			<origin xyz="0 0 -0.328" rpy="${ -M_PI / 2.0 } 0 0"/>
 			<parent link="${name}_3_link"/>
 			<child link="${name}_4_link"/>
@@ -232,5 +232,5 @@
 		<!-- J5 -->
 		<joint name="${name}_5_joint" type="revolute">
-			<origin xyz="0 0 0" rpy="1.57 0 0" />
+			<origin xyz="0 0 0" rpy="${ M_PI / 2.0 } 0 0" />
 			<parent link="${name}_4_link"/>
 			<child link="${name}_5_link"/>
@@ -241,5 +241,5 @@
 		<!-- J6 -->
 		<joint name="${name}_6_joint" type="revolute">
-			<origin xyz="0 0 -0.323" rpy="1.57 0 0" />
+			<origin xyz="0 0 -0.323" rpy="${ M_PI / 2.0 } 0 0" />
 			<parent link="${name}_5_link"/>
 			<child link="${name}_6_link"/>
@@ -250,5 +250,5 @@
 		<!-- J7-->
 		<joint name="${name}_7_joint" type="revolute">
-			<origin xyz="0 -0.1672 0" rpy="-1.57 0 0" />
+			<origin xyz="0 -0.1672 0" rpy="${ -M_PI / 2.0 } 0 0" />
 			<parent link="${name}_6_link"/>
 			<child link="${name}_7_link"/>

File: apc_description/urdf/sdh/sdh.xacro (robot description, xacro)
@@ -227,5 +227,5 @@
 		<!-- joint between sdh_palm_link and sdh_thumb_1_link -->
 		<joint name="${name}_thumb_1_joint" type="fixed">
-			<origin xyz="0 0.03811 0.0745 " rpy="0 0 -1.5708" />
+			<origin xyz="0 0.03811 0.0745 " rpy="0 0 ${ -M_PI / 2.0 }" />
 			<parent link="${name}_palm_link"/>
 			<child link="${name}_thumb_1_link"/>

Commit message: models: Change to simpler lwa4d model

File: apc_description/urdf/lwa4d/lwa4d.xacro (robot description, xacro)
@@ -48,5 +48,5 @@
 				<origin xyz="0 0 0" rpy="0 0 0" />
 				<geometry>
-					<mesh filename="package://apc_description/meshes/lwa4d/arm_1_link.dae" />
+					<mesh filename="package://apc_description/meshes/lwa4d/arm_1_link_simplified.ply" />
 				</geometry>
 				<material name="Schunk_LightGrey">
@@ -57,5 +57,5 @@
 				<origin xyz="0 0 0" rpy="0 0 0" />
 				<geometry>
-					<mesh filename="package://apc_description/meshes/lwa4d/arm_1_link.dae" />
+					<mesh filename="package://apc_description/meshes/lwa4d/arm_1_link_box.dae" />
 				</geometry>
 			</collision>
@@ -71,5 +71,5 @@
 				<origin xyz="0 0 0" rpy="0 0 0" />
 				<geometry>
-					<mesh filename="package://apc_description/meshes/lwa4d/arm_2_link.dae" />
+					<mesh filename="package://apc_description/meshes/lwa4d/arm_2_link_simplified.ply" />
 				</geometry>
 				<material name="Schunk_Black" />
@@ -78,5 +78,5 @@
 				<origin xyz="0 0 0" rpy="0 0 0" />
 				<geometry>
-					<mesh filename="package://apc_description/meshes/lwa4d/arm_2_link.dae"/>
+					<mesh filename="package://apc_description/meshes/lwa4d/arm_2_link_box.dae"/>
 				</geometry>
 			</collision>
@@ -92,5 +92,5 @@
 				<origin xyz="0 0 0" rpy="0 0 0" />
 				<geometry>
-					<mesh filename="package://apc_description/meshes/lwa4d/arm_3_link.dae" />
+					<mesh filename="package://apc_description/meshes/lwa4d/arm_3_link_simplified.ply" />
 				</geometry>
 				<material name="Schunk_LightGrey" />
@@ -99,5 +99,5 @@
 				<origin xyz="0 0 0" rpy="0 0 0" />
 				<geometry>
-					<mesh filename="package://apc_description/meshes/lwa4d/arm_3_link.dae"/>
+					<mesh filename="package://apc_description/meshes/lwa4d/arm_3_link_box.dae"/>
 				</geometry>
 			</collision>
@@ -113,5 +113,5 @@
 				<origin xyz="0 0 0" rpy="0 0 0" />
 				<geometry>
-					<mesh filename="package://apc_description/meshes/lwa4d/arm_4_link.dae" />
+					<mesh filename="package://apc_description/meshes/lwa4d/arm_4_link_simplified.ply" />
 				</geometry>
 				<material name="Schunk_Black" />
@@ -120,5 +120,5 @@
 				<origin xyz="0 0 0" rpy="0 0 0" />
 				<geometry>
-					<mesh filename="package://apc_description/meshes/lwa4d/arm_4_link.dae"/>
+					<mesh filename="package://apc_description/meshes/lwa4d/arm_4_link_box.dae"/>
 				</geometry>
 			</collision>
@@ -134,5 +134,5 @@
 				<origin xyz="0 0 0" rpy="0 0 0" />
 				<geometry>
-					<mesh filename="package://apc_description/meshes/lwa4d/arm_5_link_phys.dae" />
+					<mesh filename="package://apc_description/meshes/lwa4d/arm_5_link_phys_simplified.ply" />
 				</geometry>
 				<material name="Schunk_LightGrey" />
@@ -141,5 +141,5 @@
 				<origin xyz="0 0 0" rpy="0 0 0" />
 				<geometry>
-					<mesh filename="package://apc_description/meshes/lwa4d/arm_5_link_phys.dae"/>
+					<mesh filename="package://apc_description/meshes/lwa4d/arm_5_link_phys_box.dae"/>
 				</geometry>
 			</collision>
@@ -155,5 +155,5 @@
 				<origin xyz="0 0 0" rpy="0 0 0" />
 				<geometry>
-					<mesh filename="package://apc_description/meshes/lwa4d/arm_6_link.dae" />
+					<mesh filename="package://apc_description/meshes/lwa4d/arm_6_link_simplified.ply" />
 				</geometry>
 				<material name="Schunk_Black" />
@@ -162,5 +162,5 @@
 				<origin xyz="0 0 0" rpy="0 0 0" />
 				<geometry>
-					<mesh filename="package://apc_description/meshes/lwa4d/arm_6_link.dae"/>
+					<mesh filename="package://apc_description/meshes/lwa4d/arm_6_link_box.dae"/>
 				</geometry>
 			</collision>
@@ -176,5 +176,5 @@
 				<origin xyz="0 0 0" rpy="0 0 0" />
 				<geometry>
-					<mesh filename="package://apc_description/meshes/lwa4d/arm_7_FT_tool_changers_link.dae" />
+					<mesh filename="package://apc_description/meshes/lwa4d/arm_7_FT_tool_changers_link_simplified.ply" />
 				</geometry>
 				<material name="Schunk_LightGrey" />
@@ -183,5 +183,5 @@
 				<origin xyz="0 0 0" rpy="0 0 0" />
 				<geometry>
-					<mesh filename="package://apc_description/meshes/lwa4d/arm_7_FT_tool_changers_link.dae"/>
+					<mesh filename="package://apc_description/meshes/lwa4d/arm_7_FT_tool_changers_link_box.dae"/>
 				</geometry>
 			</collision>
