Commit message: Convert urdf to collada for trajopt

File: apc_description/urdf/crichton/crichton.urdf.xacro (robot description, xacro)
@@ -2,7 +2,7 @@
 <robot name="crichton" xmlns:xacro="http://www.ros.org/wiki/xacro">
     <!-- Include APC decriptions for LWA4 and SDH -->
-    <xacro:include filename="$(find apc_description)/urdf/lwa4d_torso/lwa4d_torso.urdf.xacro"/>
-    <xacro:include filename="$(find apc_description)/urdf/lwa4d/lwa4d.urdf.xacro" />
-    <xacro:include filename="$(find apc_description)/urdf/sdh/sdh.urdf.xacro"     />
+    <xacro:include filename="$(find apc_description)/urdf/lwa4d_torso/lwa4d_torso.xacro"/>
+    <xacro:include filename="$(find apc_description)/urdf/lwa4d/lwa4d.xacro" />
+    <xacro:include filename="$(find apc_description)/urdf/sdh/sdh.xacro"     />
     <xacro:include filename="$(find apc_description)/urdf/materials.urdf.xacro"   />
     <!-- Math constants -->

File: apc_description/urdf/lwa4d/lwa4d.urdf.xacro (robot description, xacro)
@@ -1,263 +1,13 @@
 <?xml version="1.0"?>
-<robot xmlns:xacro="http://www.ros.org/wiki/xacro">
-	<!-- Differences with lwa4d-->
-	<!-- Flip axis 2,4,6,7-->
-	<!-- Change initial distance to joint 0 from 0.1375 to 0.12 to have -->
-	<!-- pedestal distance of 0.12 + 0.18 = 0.300 -->
-	<!-- To simulate with left guy, rotate w.r.t. world 180 w.r.t. Z axis -->
-	<!-- F/T changes -->
-	<!-- December 16th, 2014 -->
-	<!-- Changed distance from J6 to Jt from 0.075 to 0.1672 (including the F/T + tool changer) -->
-	<!-- Distances from Schunk datasheet -->
-	<!-- xacro changes -->
-	<!-- December 17th, 2014 -->
-    <!-- Changed lwa4d_right_phys.urdf into a xacro macro -->
-    <xacro:include filename="$(find schunk_description)/urdf/lwa4d/lwa4d.gazebo.xacro"/>
-    <xacro:include filename="$(find schunk_description)/urdf/lwa4d/lwa4d.transmission.xacro"/>
-	<xacro:macro name="schunk_lwa4d" params="parent name *origin">
-	    <!-- L0 -->
-	    <link name="${name}_0_link">
-		    <inertial>
-				<origin xyz="0 0 0" rpy="0 0 0"/>
-				<mass value="1.0"/>
-				<inertia ixx="0.01" ixy="0" ixz="0" iyy="0.01" iyz="0" izz="0.01" />
-			</inertial>
-            <visual>
-                <origin xyz="0 0 0" rpy="0 0 0"/>
-                <geometry>
-                    <cylinder radius="0.045" length="0.03"/>
-                </geometry>
-                <material name="Schunk/Black"/>
-            </visual>
-            <collision>
-                <origin xyz="0 0 0" rpy="0 0 0"/>
-                <geometry>
-                    <cylinder radius="0.045" length="0.03"/>
-                </geometry>
-            </collision>
-		</link>
-	    <!-- L1 -->
-		<link name="${name}_1_link">
-			<inertial>
-				<origin xyz="0 0 0" rpy="0 0 0" />
-				<!--mass value="5.9907"/-->
-				<mass value="2.0"/>
-				<inertia ixx="0.01" ixy="0" ixz="0" iyy="0.01" iyz="0" izz="0.01" />
-			</inertial>
-			<visual>
-				<origin xyz="0 0 0" rpy="0 0 0" />
-				<geometry>
-					<mesh filename="package://apc_description/meshes/lwa4d/arm_1_link.dae" />
-				</geometry>
-				<material name="Schunk_LightGrey">
-					<color rgba="0.7 0.7 0.7 1.0"/>
-				</material>
-			</visual>
-			<collision>
-				<origin xyz="0 0 0" rpy="0 0 0" />
-				<geometry>
-					<mesh filename="package://apc_description/meshes/lwa4d/arm_1_link.dae" />
-				</geometry>
-			</collision>
-		</link>
-		<!-- L2 -->
-		<link name="${name}_2_link">
-			<inertial>
-				<origin xyz="0 0 0" rpy="0 0 0"/>
-				<mass value="2.0"/>
-				<inertia ixx="0.03" ixy="0" ixz="0" iyy="0.03" iyz="0" izz="0.03" />
-			</inertial>
-			<visual>
-				<origin xyz="0 0 0" rpy="0 0 0" />
-				<geometry>
-					<mesh filename="package://apc_description/meshes/lwa4d/arm_2_link.dae" />
-				</geometry>
-				<material name="Schunk_Black" />
-			</visual>
-			<collision>
-				<origin xyz="0 0 0" rpy="0 0 0" />
-				<geometry>
-					<mesh filename="package://apc_description/meshes/lwa4d/arm_2_link.dae"/>
-				</geometry>
-			</collision>
-		</link>
-		<!-- L3 -->
-		<link name="${name}_3_link">
-			<inertial>
-				<origin xyz="0 0 0" rpy="0 0 0"/>
-				<mass value="2.0"/>
-				<inertia ixx="0.03" ixy="0" ixz="0" iyy="0.03" iyz="0" izz="0.03" />
-			</inertial>
-			<visual>
-				<origin xyz="0 0 0" rpy="0 0 0" />
-				<geometry>
-					<mesh filename="package://apc_description/meshes/lwa4d/arm_3_link.dae" />
-				</geometry>
-				<material name="Schunk_LightGrey" />
-			</visual>
-			<collision>
-				<origin xyz="0 0 0" rpy="0 0 0" />
-				<geometry>
-					<mesh filename="package://apc_description/meshes/lwa4d/arm_3_link.dae"/>
-				</geometry>
-			</collision>
-		</link>
-		<!-- L4 -->
-		<link name="${name}_4_link">
-			<inertial>
-				<origin xyz="0 0 0" rpy="0 0 0"/>
-				<mass value="2.0"/>
-				<inertia ixx="0.03" ixy="0" ixz="0" iyy="0.03" iyz="0" izz="0.03" />
-			</inertial>
-			<visual>
-				<origin xyz="0 0 0" rpy="0 0 0" />
-				<geometry>
-					<mesh filename="package://apc_description/meshes/lwa4d/arm_4_link.dae" />
-				</geometry>
-				<material name="Schunk_Black" />
-			</visual>
-			<collision>
-				<origin xyz="0 0 0" rpy="0 0 0" />
-				<geometry>
-					<mesh filename="package://apc_description/meshes/lwa4d/arm_4_link.dae"/>
-				</geometry>
-			</collision>
-		</link>
-		<!-- L5 -->
-		<link name="${name}_5_link">
-			<inertial>
-				<origin xyz="0 0 0" rpy="0 0 0"/>
-				<mass value="2.313272"/>
-				<inertia ixx="0.03" ixy="0" ixz="0" iyy="0.03" iyz="0" izz="0.03" />
-			</inertial>
-			<visual>
-				<origin xyz="0 0 0" rpy="0 0 0" />
-				<geometry>
-					<mesh filename="package://apc_description/meshes/lwa4d/arm_5_link_phys.dae" />
-				</geometry>
-				<material name="Schunk_LightGrey" />
-			</visual>
-			<collision>
-				<origin xyz="0 0 0" rpy="0 0 0" />
-				<geometry>
-					<mesh filename="package://apc_description/meshes/lwa4d/arm_5_link_phys.dae"/>
-				</geometry>
-			</collision>
-		</link>
-		<!-- L6 -->
-		<link name="${name}_6_link">
-			<inertial>
-				<origin xyz="0 0 0" rpy="0 0 0"/>
-				<mass value="2.057856"/>
-				<inertia ixx="0.01" ixy="0" ixz="0" iyy="0.01" iyz="0" izz="0.01" />
-			</inertial>
-			<visual>
-				<origin xyz="0 0 0" rpy="0 0 0" />
-				<geometry>
-					<mesh filename="package://apc_description/meshes/lwa4d/arm_6_link.dae" />
-				</geometry>
-				<material name="Schunk_Black" />
-			</visual>
-			<collision>
-				<origin xyz="0 0 0" rpy="0 0 0" />
-				<geometry>
-					<mesh filename="package://apc_description/meshes/lwa4d/arm_6_link.dae"/>
-				</geometry>
-			</collision>
-		</link>
-		<!-- L7-->
-		<link name="${name}_7_link">
-			<inertial>
-				<origin xyz="0 0 0" rpy="0 0 0"/>
-				<mass value="1.120198"/>
-				<inertia ixx="0.01" ixy="0" ixz="0" iyy="0.01" iyz="0" izz="0.01" />
-			</inertial>
-			<visual>
-				<origin xyz="0 0 0" rpy="0 0 0" />
-				<geometry>
-					<mesh filename="package://apc_description/meshes/lwa4d/arm_7_FT_tool_changers_link.dae" />
-				</geometry>
-				<material name="Schunk_LightGrey" />
-			</visual>
-			<collision>
-				<origin xyz="0 0 0" rpy="0 0 0" />
-				<geometry>
-					<mesh filename="package://apc_description/meshes/lwa4d/arm_7_FT_tool_changers_link.dae"/>
-				</geometry>
-			</collision>
-		</link>
-	    <!-- J0 -->
-	    <joint name="${name}_0_joint" type="fixed" >
-            <xacro:insert_block name="origin"/>
-		    <parent link="${parent}" />
-		    <child link="${name}_0_link" />
-	    </joint>
-	    <!-- J1 -->
-		<joint name="${name}_1_joint" type="revolute">
-			<!-- <origin xyz="0 0.1375 0" rpy="1.57 3.1416 0"/> -->
-			<origin xyz="0 0.12 0" rpy="1.57 3.1416 0"/>
-			<parent link="${name}_0_link"/>
-			<child link="${name}_1_link"/>
-			<axis xyz="0 0 1"/>
-			<dynamics damping="10" />
-			<limit effort="370" velocity="2.0" lower="-3.14" upper="3.14"/>
-		</joint>
-	    <!-- J2 -->
-		<joint name="${name}_2_joint" type="revolute">
-			<origin xyz="0 0 -0.18" rpy="-1.57 0 0"/>
-			<parent link="${name}_1_link"/>
-			<child link="${name}_2_link"/>
-			<axis xyz="0 0 -1"/>
-			<dynamics damping="10" />
-			<limit effort="370" velocity="2.0" lower="-1.97" upper="1.97"/>
-		</joint>
-		<!-- J3-->
-		<joint name="${name}_3_joint" type="revolute">
-			<origin xyz="0 0 0" rpy="1.57 0 0"/>
-			<parent link="${name}_2_link"/>
-			<child link="${name}_3_link"/>
-			<axis xyz="0 0 1"/>
-			<dynamics damping="5" />
-			<limit effort="176" velocity="2.0" lower="-3.14" upper="3.14"/>
-		</joint>
-		<!-- J4 -->
-		<joint name="${name}_4_joint" type="revolute">
-			<origin xyz="0 0 -0.328" rpy="-1.57 0 0"/>
-			<parent link="${name}_3_link"/>
-			<child link="${name}_4_link"/>
-			<axis xyz="0 0 -1" />
-			<dynamics damping="5" />
-			<limit effort="176" velocity="2.0" lower="-2.08208" upper="2.08208"/>
-		</joint>
-		<!-- J5 -->
-		<joint name="${name}_5_joint" type="revolute">
-			<origin xyz="0 0 0" rpy="1.57 0 0" />
-			<parent link="${name}_4_link"/>
-			<child link="${name}_5_link"/>
-			<axis xyz="0 0 1" />
-			<dynamics damping="5" />
-			<limit effort="41.6" velocity="2.0" lower="-3.14" upper="3.14" />
-		</joint>
-		<!-- J6 -->
-		<joint name="${name}_6_joint" type="revolute">
-			<origin xyz="0 0 -0.323" rpy="1.57 0 0" />
-			<parent link="${name}_5_link"/>
-			<child link="${name}_6_link"/>
-			<axis xyz="0 0 -1" />
-			<dynamics damping="5" />
-			<limit effort="20.1" velocity="2.0" lower="-1.8" upper="1.8" />
-		</joint>
-		<!-- J7-->
-		<joint name="${name}_7_joint" type="revolute">
-			<origin xyz="0 -0.1672 0" rpy="-1.57 0 0" />
-			<parent link="${name}_6_link"/>
-			<child link="${name}_7_link"/>
-			<axis xyz="0 0 -1" />
-			<dynamics damping="5" />
-			<limit effort="9.6" velocity="2.0" lower="-3.14" upper="3.14" />
-		</joint>
-        <!-- extensions -->
-        <xacro:schunk_lwa4d_gazebo name="${name}"/>
-        <xacro:schunk_lwa4d_transmission name="${name}"/>
-    </xacro:macro>
+<robot name="lwa4d" xmlns:xacro="http://www.ros.org/wiki/xacro">
+    <!-- Include decriptions for SDH -->
+    <xacro:include filename="$(find apc_description)/urdf/lwa4d/lwa4d.xacro" />
+    <!-- Math constants -->
+    <xacro:property name="M_PI" value="3.141592653" />
+    <!-- LWA4D origin. -->
+    <link name="lwa4d_origin" />
+    <!-- Assemble LWA4D -->
+    <xacro:schunk_lwa4d parent="lwa4d_origin" name="lwa4d_arm" >
+        <origin xyz="0 0 0" rpy="0 0 0" />
+    </xacro:schunk_lwa4d>
 </robot>

File: apc_description/urdf/lwa4d_torso/lwa4d_torso.urdf.xacro (robot description, xacro)
@@ -1,52 +1,13 @@
 <?xml version="1.0"?>
-<robot xmlns:xacro="http://www.ros.org/wiki/xacro">
-	<xacro:macro name="schunk_lwa4d_torso" params="parent name *origin">
-		<link name="${name}_vertical_support">
-			<inertial>
-				<origin xyz="0.0 0.0 0.0" rpy="0 0 0"/>
-				<mass value="5.0"/>
-				<inertia ixx="1" ixy="0.0" ixz="0.0" iyy="1" iyz="0.0" izz="1" />
-			</inertial>
-			<visual>
-				<origin xyz="-0.45 -0.45 0.0" rpy="0 0 0"/>
-				<geometry>
-					<mesh filename="package://apc_description/meshes/lwa4d_torso/vertical_support.dae" scale="1 1 1" />
-				</geometry>
-			</visual>
-			<collision>
-				<origin xyz="-0.45 -0.45 0.0" rpy="0 0 0"/>
-				<geometry>
-					<mesh filename="package://apc_description/meshes/lwa4d_torso/vertical_support.dae" scale="1 1 1" />
-				</geometry>
-			</collision>
-		</link>
-		<joint name="${name}_base_joint" type="fixed">
-			<xacro:insert_block name="origin"/>
-			<parent link="${parent}" />
-			<child  link="${name}_vertical_support" />
-		</joint>
-		<link name="${name}_middle_support">
-			<inertial>
-				<origin xyz="0.0 0.0 0.0" rpy="0 0 0"/>
-				<mass value="5.0"/>
-				<inertia ixx="1" ixy="0.0" ixz="0.0" iyy="1" iyz="0.0" izz="1" />
-			</inertial>
-			<visual>
-				<geometry>
-					<mesh filename="package://apc_description/meshes/lwa4d_torso/middle_support.dae" scale="1 1 1" />
-				</geometry>
-			</visual>
-			<collision>
-				<geometry>
-					<mesh filename="package://apc_description/meshes/lwa4d_torso/middle_support.dae" scale="1 1 1" />
-				</geometry>
-			</collision>
-		</link>
-		<!-- TODO Turn into revolute joint -->
-		<joint name="${name}_torso_joint" type="fixed">
-			<origin xyz="0 0 1.23" rpy="0 0 0" />
-			<parent link="${name}_vertical_support" />
-			<child  link="${name}_middle_support" />
-		</joint>
-	</xacro:macro>
+<robot name="lwa4d_torso" xmlns:xacro="http://www.ros.org/wiki/xacro">
+    <!-- Include decriptions for LWA4D_TORSO -->
+    <xacro:include filename="$(find apc_description)/urdf/lwa4d_torso/lwa4d_torso.xacro" />
+    <!-- Math constants -->
+    <xacro:property name="M_PI" value="3.141592653" />
+    <!-- LWA4D_TORSO origin. -->
+    <link name="lwa4d_torso_origin" />
+    <!-- Assemble LWA4D_TORSO hand -->
+    <xacro:schunk_lwa4d_torso parent="lwa4d_torso_origin" name="lwa4d_torso" >
+        <origin xyz="0 0 0" rpy="0 0 0" />
+    </xacro:schunk_lwa4d_torso>
 </robot>
