Commit message: WIP Add crichton torso joint

File: apc_description/urdf/lwa4d_torso/lwa4d_torso.xacro (robot description, xacro)
@@ -44,8 +44,11 @@
 		</link>
 		<!-- TODO Turn into revolute joint -->
-		<joint name="${name}_torso_joint" type="fixed">
+		<joint name="${name}_torso_joint" type="revolute">
 			<origin xyz="0 0 1.23" rpy="0 0 0" />
 			<parent link="${name}_vertical_support" />
 			<child  link="${name}_middle_support" />
+			<axis xyz="0 0 -1" />
+			<dynamics damping="5" />
+			<limit effort="20.1" velocity="2.0" lower="-1.8" upper="1.8" />
 		</joint>
 	</xacro:macro>

Commit message: models: Add bottom and top kinect models

File: apc_description/urdf/lwa4d_torso/lwa4d_torso.xacro (robot description, xacro)
@@ -2,4 +2,5 @@
 <robot name="lwa4d_torso" xmlns:xacro="http://www.ros.org/wiki/xacro">
 	<xacro:macro name="schunk_lwa4d_torso" params="parent name *origin">
+	<xacro:property name="M_PI" value="3.141592653" />
 		<link name="${name}_vertical_support">
 			<inertial>
@@ -52,4 +53,48 @@
 			<limit effort="20.1" velocity="2.0" lower="-1.8" upper="1.8" />
 		</joint>
+		<link name="${name}_top_kinect">
+			<inertial>
+				<origin xyz="0.0 0.0 0.0" rpy="0 0 0"/>
+				<mass value="5.0"/>
+				<inertia ixx="1" ixy="0.0" ixz="0.0" iyy="1" iyz="0.0" izz="1" />
+			</inertial>
+			<visual>
+				<geometry>
+					<mesh filename="package://apc_description/meshes/lwa4d_torso/top_kinect.dae" scale="1 1 1" />
+				</geometry>
+			</visual>
+			<collision>
+				<geometry>
+					<mesh filename="package://apc_description/meshes/lwa4d_torso/top_kinect.dae" scale="1 1 1" />
+				</geometry>
+			</collision>
+		</link>
+		<joint name="${name}_top_kinect_joint" type="fixed">
+			<origin xyz="0 0 0.055" rpy="0 0 ${M_PI/2}" />
+			<parent link="${name}_middle_support" />
+			<child  link="${name}_top_kinect" />
+		</joint>
+		<link name="${name}_bottom_kinect">
+			<inertial>
+				<origin xyz="0.0 0.0 0.0" rpy="0 0 0"/>
+				<mass value="5.0"/>
+				<inertia ixx="1" ixy="0.0" ixz="0.0" iyy="1" iyz="0.0" izz="1" />
+			</inertial>
+			<visual>
+				<geometry>
+					<mesh filename="package://apc_description/meshes/lwa4d_torso/bottom_kinect.dae" scale="1 1 1" />
+				</geometry>
+			</visual>
+			<collision>
+				<geometry>
+					<mesh filename="package://apc_description/meshes/lwa4d_torso/bottom_kinect.dae" scale="1 1 1" />
+				</geometry>
+			</collision>
+		</link>
+		<joint name="${name}_bottom_kinect_joint" type="fixed">
+			<origin xyz="-0.093 0 -0.1" rpy="0 ${M_PI} ${M_PI/2}" />
+			<parent link="${name}_middle_support" />
+			<child  link="${name}_bottom_kinect" />
+		</joint>
 	</xacro:macro>
 </robot>
